File: pcb/battleship_pcb/battleship_pcb.kicad_sch (KiCad schematic)
At the start: 56 parts, among them SW1 SW_Push, SW10 SW_Push, SW11 SW_Push, SW12 SW_Push, SW2 SW_Push, SW3 SW_Push, SW4 SW_Push, SW5 SW_Push, SW6 SW_Push, SW7 SW_Push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

Commit message: Updated kicad schematic
Connections:
- net at D1.1 (RK), D2.1 (RK): now also MC1. (PF11)
- net at D1.3 (BK), D2.3 (BK): now also MC1. (PF11)
- net at D1.4 (GK), D2.4 (GK): now also MC1. (PF11)
- net at D3.1 (RK), D4.1 (RK): now also MC2. (PF11)
- net at D3.3 (BK), D4.3 (BK): now also MC2. (PF11)
- net at D3.4 (GK), D4.4 (GK): now also MC2. (PF11)
- new net: LCD1. (VCC), MC1. (PF11) (x5)
- new net: LCD2. (VCC), MC2. (PF11) (x5)
- new net: MC1. (PF11), MC2. (PF11) (x3)
Other:
- moved on the sheet: D3, D4, LCD2, MC2
